Commit message: Add bot_drive

File: src/piyabot/bot_description/urdf/piyabot_delta.urdf.xacro (robot description, xacro)
@@ -138,7 +138,7 @@
     <origin xyz="0 0 ${chassisHeight + rplidarSize/4}" rpy="0 0 0"/>
     <parent link="chassis"/>
-    <child link="rplidar"/>
-  </joint>
-  <link name="rplidar">
+    <child link="laser"/>
+  </joint>
+  <link name="laser">
     <collision>
       <origin xyz="0 0 0" rpy="0 0 0"/>
